Commit message: Move from manual moveit to scripted python (#19)
* ruff

* move entry point in bringup

* install moveit py

* rename

* update rviz

* update description urdf and srdf

* add a cube in scene

* add gripper

* replace build and start with run.sh

* delete a file

* run

* update

* rviz

* c

* c

* c

* code

* red cube

* Add CLAUDE.md for team collaboration context

Provides project overview, goals, and key file locations for AI-assisted
development. Enables consistent context across team members.

Co-Authored-By: Claude Sonnet 4.5 <noreply@anthropic.com>

* Add volume mount for Claude data persistence

Persists /root/.claude/ directory across container rebuilds to preserve
chat history, project memory, and credentials.

* devcontainer

* script that can send to the arm to move to cube blue

* claude

* Fix CONTROL_FAILED error: mimic joint + controller config fixes

The arm motion (`move_to_cube --cube blue`) was failing with MoveIt
error -4 (CONTROL_FAILED) due to multiple cascading controller issues.

Root cause: `robotic_arm.ros2_control.xacro` (MoveIt's hardware config)
gave `right_finger_joint` a command_interface, which conflicts with the
URDF <mimic> tag — ROS2 Jazzy enforces that mimic joints cannot have
command interfaces, crashing the controller_manager at startup.

Fixes:
- Remove command_interface from right_finger_joint in ros2_control.xacro
- Remove deprecated <param name="mimic"> from URDF ros2_control section
  (Jazzy reads mimic info from standard URDF <mimic> tag only)
- Remove duplicate controller_manager from launch file (demo.launch.py
  already starts one)
- Fix gripper_controller indentation in moveit_controllers.yaml
- Fix ros2_controllers.yaml: add trajectory constraints, remove velocity
  state_interface (URDF only exports position)
- Add diagnostic logging: controller status, trajectory waypoints,
  human-readable MoveIt error codes

Co-Authored-By: Claude Opus 4.6 <noreply@anthropic.com>

* The script is working

---------

Co-authored-by: Daniel Iacob <daniel_iacob>
Co-authored-by: Claude Sonnet 4.5 <noreply@anthropic.com>

File: src/robotic_arm_description/urdf/robotic_arm.urdf.xacro (robot description, xacro)
@@ -31,9 +31,8 @@
       <material name="orange"/>
     </visual>
-    <visual>
-      <origin xyz="0 0 0.1" rpy="${pi/2} 0 0"/>
-      <geometry><cylinder length="0.15" radius="0.06"/></geometry>
-      <material name="dark_grey"/>
-    </visual>
+    <collision>
+      <origin xyz="0 0 0.05" rpy="0 0 0"/>
+      <geometry><cylinder length="0.1" radius="0.08"/></geometry>
+    </collision>
   </link>
   <joint name="joint_2" type="revolute">
@@ -50,9 +49,8 @@
       <material name="silver"/>
     </visual>
-    <visual>
-      <origin xyz="0 0 0.4" rpy="${pi/2} 0 0"/>
-      <geometry><cylinder length="0.1" radius="0.05"/></geometry>
-      <material name="dark_grey"/>
-    </visual>
+    <collision>
+      <origin xyz="0 0 0.2" rpy="0 0 0"/>
+      <geometry><box size="0.06 0.06 0.4"/></geometry>
+    </collision>
   </link>
   <joint name="joint_3" type="revolute">
@@ -69,5 +67,62 @@
       <material name="orange"/>
     </visual>
+    <collision>
+      <origin xyz="0 0 0.15" rpy="0 0 0"/>
+      <geometry><cylinder length="0.3" radius="0.03"/></geometry>
+    </collision>
   </link>
+  <joint name="gripper_base_joint" type="fixed">
+    <parent link="forearm"/>
+    <child link="gripper_base"/>
+    <origin xyz="0 0 0.3" rpy="0 0 0"/>
+  </joint>
+  <link name="gripper_base">
+    <visual>
+      <geometry><box size="0.1 0.1 0.05"/></geometry>
+      <material name="dark_grey"/>
+    </visual>
+    <collision>
+      <geometry><box size="0.1 0.1 0.05"/></geometry>
+    </collision>
+  </link>
+  <joint name="left_finger_joint" type="prismatic">
+    <parent link="gripper_base"/>
+    <child link="left_finger"/>
+    <origin xyz="0 0.04 0.05" rpy="0 0 0"/>
+    <axis xyz="0 1 0"/>
+    <limit lower="-0.04" upper="0.0" effort="10.0" velocity="0.1"/>
+  </joint>
+  <link name="left_finger">
+    <visual>
+      <geometry><box size="0.02 0.02 0.08"/></geometry>
+      <material name="silver"/>
+    </visual>
+    <collision>
+      <geometry><box size="0.02 0.02 0.08"/></geometry>
+    </collision>
+  </link>
+  <joint name="right_finger_joint" type="prismatic">
+    <parent link="gripper_base"/>
+    <child link="right_finger"/>
+    <origin xyz="0 -0.04 0.05" rpy="0 0 0"/>
+    <axis xyz="0 1 0"/>
+    <limit lower="0.0" upper="0.04" effort="10.0" velocity="0.1"/>
+    <mimic joint="left_finger_joint" multiplier="-1.0" offset="0.0"/>
+  </joint>
+  <link name="right_finger">
+    <visual>
+      <geometry><box size="0.02 0.02 0.08"/></geometry>
+      <material name="silver"/>
+    </visual>
+    <collision>
+      <geometry><box size="0.02 0.02 0.08"/></geometry>
+    </collision>
+  </link>
+  <link name="grasp_link"/>
+  <joint name="grasp_link_joint" type="fixed">
+    <parent link="gripper_base"/>
+    <child link="grasp_link"/>
+    <origin xyz="0 0 0.08" rpy="0 0 0"/>
+  </joint>
   <ros2_control name="RoboticArmHardware" type="system">
     <hardware><plugin>mock_components/GenericSystem</plugin></hardware>
@@ -81,4 +136,10 @@
       <command_interface name="position"/><state_interface name="position"/>
     </joint>
+    <joint name="left_finger_joint">
+      <command_interface name="position"/><state_interface name="position"/>
+    </joint>
+    <joint name="right_finger_joint">
+      <state_interface name="position"/>
+    </joint>
   </ros2_control>
 </robot>

File: src/robotic_arm_moveit_config/config/robotic_arm.ros2_control.xacro (robot description, xacro)
@@ -5,5 +5,4 @@
         <ros2_control name="${name}" type="system">
             <hardware>
-                <!-- By default, set up controllers for simulation. This won't work on real hardware -->
                 <plugin>mock_components/GenericSystem</plugin>
             </hardware>
@@ -13,5 +12,4 @@
                   <param name="initial_value">${initial_positions['joint_1']}</param>
                 </state_interface>
-                <state_interface name="velocity"/>
             </joint>
             <joint name="joint_2">
@@ -20,5 +18,4 @@
                   <param name="initial_value">${initial_positions['joint_2']}</param>
                 </state_interface>
-                <state_interface name="velocity"/>
             </joint>
             <joint name="joint_3">
@@ -27,5 +24,15 @@
                   <param name="initial_value">${initial_positions['joint_3']}</param>
                 </state_interface>
-                <state_interface name="velocity"/>
+            </joint>
+            <joint name="left_finger_joint">
+                <command_interface name="position"/>
+                <state_interface name="position">
+                  <param name="initial_value">0.0</param>
+                </state_interface>
+            </joint>
+            <joint name="right_finger_joint">
+                <state_interface name="position">
+                  <param name="initial_value">0.0</param>
+                </state_interface>
             </joint>
         </ros2_control>
