Commit message: urdf add ros control tags

File: src/robotic_arm_description/urdf/robotic_arm.urdf.xacro (robot description, xacro)
@@ -31,5 +31,7 @@
     <parent link="link_1"/>
     <child link="link_2"/>
-    <origin xyz="0 0 0.4" rpy="0 0 0"/> <axis xyz="0 1 0"/>               <limit lower="-1.57" upper="1.57" effort="10.0" velocity="1.0"/>
+    <origin xyz="0 0 0.4" rpy="0 0 0"/>
+    <axis xyz="0 1 0"/>
+    <limit lower="-1.57" upper="1.57" effort="10.0" velocity="1.0"/>
   </joint>
   <link name="link_2">
@@ -44,3 +46,20 @@
     </visual>
   </link>
+  <ros2_control name="RoboticArmHardware" type="system">
+    <hardware>
+      <plugin>mock_components/GenericSystem</plugin>
+    </hardware>
+    <joint name="joint_1">
+      <command_interface name="position"/>
+      <state_interface name="position">
+        <param name="initial_value">0.0</param>
+      </state_interface>
+    </joint>
+    <joint name="joint_2">
+      <command_interface name="position"/>
+      <state_interface name="position">
+        <param name="initial_value">0.0</param>
+      </state_interface>
+    </joint>
+  </ros2_control>
 </robot>

Commit message: Improve robot urdf

File: src/robotic_arm_description/urdf/robotic_arm.urdf.xacro (robot description, xacro)
@@ -1,64 +1,83 @@
 <?xml version="1.0"?>
 <robot xmlns:xacro="http://www.ros.org/wiki/xacro" name="robotic_arm">
+  <material name="dark_grey"><color rgba="0.2 0.2 0.2 1"/></material>
+  <material name="orange"><color rgba="1.0 0.5 0 1"/></material>
+  <material name="silver"><color rgba="0.8 0.8 0.8 1"/></material>
+  <link name="world"/>
+  <joint name="world_joint" type="fixed">
+    <parent link="world"/>
+    <child link="base_link"/>
+    <origin xyz="0 0 0" rpy="0 0 0"/>
+  </joint>
   <link name="base_link">
     <visual>
-      <geometry>
-        <cylinder length="0.05" radius="0.1"/>
-      </geometry>
-      <material name="blue">
-        <color rgba="0 0 1 1"/>
-      </material>
+      <geometry><cylinder length="0.1" radius="0.12"/></geometry>
+      <material name="dark_grey"/>
     </visual>
+    <collision>
+      <geometry><cylinder length="0.1" radius="0.12"/></geometry>
+    </collision>
   </link>
   <joint name="joint_1" type="continuous">
     <parent link="base_link"/>
-    <child link="link_1"/>
+    <child link="shoulder_link"/>
     <origin xyz="0 0 0.05" rpy="0 0 0"/>
     <axis xyz="0 0 1"/>
   </joint>
-  <link name="link_1">
+  <link name="shoulder_link">
     <visual>
-      <origin xyz="0 0 0.2" rpy="0 0 0"/>
-      <geometry>
-        <box size="0.05 0.05 0.4"/>
-      </geometry>
-      <material name="red">
-        <color rgba="1 0 0 1"/>
-      </material>
+      <origin xyz="0 0 0.05" rpy="0 0 0"/>
+      <geometry><cylinder length="0.1" radius="0.08"/></geometry>
+      <material name="orange"/>
+    </visual>
+    <visual>
+      <origin xyz="0 0 0.1" rpy="${pi/2} 0 0"/>
+      <geometry><cylinder length="0.15" radius="0.06"/></geometry>
+      <material name="dark_grey"/>
     </visual>
   </link>
   <joint name="joint_2" type="revolute">
-    <parent link="link_1"/>
-    <child link="link_2"/>
+    <parent link="shoulder_link"/>
+    <child link="upper_arm"/>
+    <origin xyz="0 0 0.1" rpy="0 0 0"/>
+    <axis xyz="0 1 0"/>
+    <limit lower="-1.57" upper="1.57" effort="50.0" velocity="1.0"/>
+  </joint>
+  <link name="upper_arm">
+    <visual>
+      <origin xyz="0 0 0.2" rpy="0 0 0"/>
+      <geometry><box size="0.06 0.06 0.4"/></geometry>
+      <material name="silver"/>
+    </visual>
+    <visual>
+      <origin xyz="0 0 0.4" rpy="${pi/2} 0 0"/>
+      <geometry><cylinder length="0.1" radius="0.05"/></geometry>
+      <material name="dark_grey"/>
+    </visual>
+  </link>
+  <joint name="joint_3" type="revolute">
+    <parent link="upper_arm"/>
+    <child link="forearm"/>
     <origin xyz="0 0 0.4" rpy="0 0 0"/>
     <axis xyz="0 1 0"/>
-    <limit lower="-1.57" upper="1.57" effort="10.0" velocity="1.0"/>
+    <limit lower="-2.0" upper="2.0" effort="30.0" velocity="1.5"/>
   </joint>
-  <link name="link_2">
+  <link name="forearm">
     <visual>
       <origin xyz="0 0 0.15" rpy="0 0 0"/>
-      <geometry>
-        <box size="0.04 0.04 0.3"/>
-      </geometry>
-      <material name="green">
-        <color rgba="0 1 0 1"/>
-      </material>
+      <geometry><cylinder length="0.3" radius="0.03"/></geometry>
+      <material name="orange"/>
     </visual>
   </link>
   <ros2_control name="RoboticArmHardware" type="system">
-    <hardware>
-      <plugin>mock_components/GenericSystem</plugin>
-    </hardware>
+    <hardware><plugin>mock_components/GenericSystem</plugin></hardware>
     <joint name="joint_1">
-      <command_interface name="position"/>
-      <state_interface name="position">
-        <param name="initial_value">0.0</param>
-      </state_interface>
+      <command_interface name="position"/><state_interface name="position"/>
     </joint>
     <joint name="joint_2">
-      <command_interface name="position"/>
-      <state_interface name="position">
-        <param name="initial_value">0.0</param>
-      </state_interface>
+      <command_interface name="position"/><state_interface name="position"/>
+    </joint>
+    <joint name="joint_3">
+      <command_interface name="position"/><state_interface name="position"/>
     </joint>
   </ros2_control>

Commit message: update description urdf and srdf

File: src/robotic_arm_description/urdf/robotic_arm.urdf.xacro (robot description, xacro)
@@ -31,9 +31,8 @@
       <material name="orange"/>
     </visual>
-    <visual>
-      <origin xyz="0 0 0.1" rpy="${pi/2} 0 0"/>
-      <geometry><cylinder length="0.15" radius="0.06"/></geometry>
-      <material name="dark_grey"/>
-    </visual>
+    <collision>
+      <origin xyz="0 0 0.05" rpy="0 0 0"/>
+      <geometry><cylinder length="0.1" radius="0.08"/></geometry>
+    </collision>
   </link>
   <joint name="joint_2" type="revolute">
@@ -50,9 +49,8 @@
       <material name="silver"/>
     </visual>
-    <visual>
-      <origin xyz="0 0 0.4" rpy="${pi/2} 0 0"/>
-      <geometry><cylinder length="0.1" radius="0.05"/></geometry>
-      <material name="dark_grey"/>
-    </visual>
+    <collision>
+      <origin xyz="0 0 0.2" rpy="0 0 0"/>
+      <geometry><box size="0.06 0.06 0.4"/></geometry>
+    </collision>
   </link>
   <joint name="joint_3" type="revolute">
@@ -69,4 +67,8 @@
       <material name="orange"/>
     </visual>
+    <collision>
+      <origin xyz="0 0 0.15" rpy="0 0 0"/>
+      <geometry><cylinder length="0.3" radius="0.03"/></geometry>
+    </collision>
   </link>
   <ros2_control name="RoboticArmHardware" type="system">

Commit message: add gripper

File: src/robotic_arm_description/urdf/robotic_arm.urdf.xacro (robot description, xacro)
@@ -72,4 +72,51 @@
     </collision>
   </link>
+  <joint name="gripper_base_joint" type="fixed">
+    <parent link="forearm"/>
+    <child link="gripper_base"/>
+    <origin xyz="0 0 0.3" rpy="0 0 0"/>
+  </joint>
+  <link name="gripper_base">
+    <visual>
+      <geometry><box size="0.1 0.1 0.05"/></geometry>
+      <material name="dark_grey"/>
+    </visual>
+    <collision>
+      <geometry><box size="0.1 0.1 0.05"/></geometry>
+    </collision>
+  </link>
+  <joint name="left_finger_joint" type="prismatic">
+    <parent link="gripper_base"/>
+    <child link="left_finger"/>
+    <origin xyz="0 0.04 0.05" rpy="0 0 0"/>
+    <axis xyz="0 1 0"/>
+    <limit lower="-0.04" upper="0.0" effort="10.0" velocity="0.1"/>
+  </joint>
+  <link name="left_finger">
+    <visual>
+      <geometry><box size="0.02 0.02 0.08"/></geometry>
+      <material name="silver"/>
+    </visual>
+    <collision>
+      <geometry><box size="0.02 0.02 0.08"/></geometry>
+    </collision>
+  </link>
+  <joint name="right_finger_joint" type="prismatic">
+    <parent link="gripper_base"/>
+    <child link="right_finger"/>
+    <origin xyz="0 -0.04 0.05" rpy="0 0 0"/>
+    <axis xyz="0 1 0"/>
+    <limit lower="0.0" upper="0.04" effort="10.0" velocity="0.1"/>
+    <mimic joint="left_finger_joint" multiplier="-1.0" offset="0.0"/>
+  </joint>
+  <link name="right_finger">
+    <visual>
+      <geometry><box size="0.02 0.02 0.08"/></geometry>
+      <material name="silver"/>
+    </visual>
+    <collision>
+      <geometry><box size="0.02 0.02 0.08"/></geometry>
+    </collision>
+  </link>
   <ros2_control name="RoboticArmHardware" type="system">
     <hardware><plugin>mock_components/GenericSystem</plugin></hardware>
@@ -83,4 +130,10 @@
       <command_interface name="position"/><state_interface name="position"/>
     </joint>
+    <joint name="left_finger_joint">
+      <command_interface name="position"/><state_interface name="position"/>
+    </joint>
+    <joint name="right_finger_joint">
+      <command_interface name="position"/><state_interface name="position"/>
+    </joint>
   </ros2_control>
 </robot>

File: src/robotic_arm_moveit_config/config/robotic_arm.ros2_control.xacro (robot description, xacro)
@@ -5,5 +5,4 @@
         <ros2_control name="${name}" type="system">
             <hardware>
-                <!-- By default, set up controllers for simulation. This won't work on real hardware -->
                 <plugin>mock_components/GenericSystem</plugin>
             </hardware>
@@ -13,5 +12,4 @@
                   <param name="initial_value">${initial_positions['joint_1']}</param>
                 </state_interface>
-                <state_interface name="velocity"/>
             </joint>
             <joint name="joint_2">
@@ -20,5 +18,4 @@
                   <param name="initial_value">${initial_positions['joint_2']}</param>
                 </state_interface>
-                <state_interface name="velocity"/>
             </joint>
             <joint name="joint_3">
@@ -27,5 +24,16 @@
                   <param name="initial_value">${initial_positions['joint_3']}</param>
                 </state_interface>
-                <state_interface name="velocity"/>
+            </joint>
+            <joint name="left_finger_joint">
+                <command_interface name="position"/>
+                <state_interface name="position">
+                  <param name="initial_value">0.0</param>
+                </state_interface>
+            </joint>
+            <joint name="right_finger_joint">
+                <command_interface name="position"/>
+                <state_interface name="position">
+                  <param name="initial_value">0.0</param>
+                </state_interface>
             </joint>
         </ros2_control>

Commit message: update

File: src/robotic_arm_description/urdf/robotic_arm.urdf.xacro (robot description, xacro)
@@ -119,4 +119,10 @@
     </collision>
   </link>
+  <link name="grasp_link"/>
+  <joint name="grasp_link_joint" type="fixed">
+    <parent link="gripper_base"/>
+    <child link="grasp_link"/>
+    <origin xyz="0 0 0.08" rpy="0 0 0"/>
+  </joint>
   <ros2_control name="RoboticArmHardware" type="system">
     <hardware><plugin>mock_components/GenericSystem</plugin></hardware>
@@ -134,5 +140,7 @@
     </joint>
     <joint name="right_finger_joint">
-      <command_interface name="position"/><state_interface name="position"/>
+      <param name="mimic">left_finger_joint</param>
+      <param name="multiplier">-1.0</param>
+      <state_interface name="position"/>
     </joint>
   </ros2_control>

Commit message: update robot urdf

File: src/robotic_arm_description/urdf/robotic_arm.urdf.xacro (robot description, xacro)
@@ -31,4 +31,8 @@
       <material name="orange"/>
     </visual>
+    <visual>
+      <geometry><sphere radius="0.065"/></geometry>
+      <material name="orange"/>
+    </visual>
     <collision>
       <origin xyz="0 0 0.05" rpy="0 0 0"/>
@@ -46,10 +50,14 @@
     <visual>
       <origin xyz="0 0 0.2" rpy="0 0 0"/>
-      <geometry><box size="0.06 0.06 0.4"/></geometry>
+      <geometry><cylinder length="0.4" radius="0.055"/></geometry>
+      <material name="silver"/>
+    </visual>
+    <visual>
+      <geometry><sphere radius="0.06"/></geometry>
       <material name="silver"/>
     </visual>
     <collision>
       <origin xyz="0 0 0.2" rpy="0 0 0"/>
-      <geometry><box size="0.06 0.06 0.4"/></geometry>
+      <geometry><cylinder length="0.4" radius="0.055"/></geometry>
     </collision>
   </link>
@@ -65,4 +73,8 @@
       <origin xyz="0 0 0.15" rpy="0 0 0"/>
       <geometry><cylinder length="0.3" radius="0.03"/></geometry>
+      <material name="orange"/>
+    </visual>
+    <visual>
+      <geometry><sphere radius="0.04"/></geometry>
       <material name="orange"/>
     </visual>

Commit message: robot visuals update

File: src/robotic_arm_description/urdf/robotic_arm.urdf.xacro (robot description, xacro)
@@ -1,7 +1,11 @@
 <?xml version="1.0"?>
 <robot xmlns:xacro="http://www.ros.org/wiki/xacro" name="robotic_arm">
-  <material name="dark_grey"><color rgba="0.2 0.2 0.2 1"/></material>
-  <material name="orange"><color rgba="1.0 0.5 0 1"/></material>
-  <material name="silver"><color rgba="0.8 0.8 0.8 1"/></material>
+  <!-- Kuka-style orange gradient base → fingers -->
+  <material name="c1"><color rgba="0.70 0.25 0.00 1"/></material>  <!-- base      — deep orange -->
+  <material name="c2"><color rgba="0.80 0.35 0.00 1"/></material>  <!-- shoulder  -->
+  <material name="c3"><color rgba="0.88 0.45 0.00 1"/></material>  <!-- upper arm -->
+  <material name="c4"><color rgba="0.94 0.55 0.05 1"/></material>  <!-- forearm   -->
+  <material name="c5"><color rgba="0.18 0.18 0.18 1"/></material>  <!-- wrist     — dark -->
+  <material name="c6"><color rgba="0.28 0.28 0.28 1"/></material>  <!-- fingers   — dark grey -->
   <link name="world"/>
   <joint name="world_joint" type="fixed">
@@ -10,8 +14,15 @@
     <origin xyz="0 0 0" rpy="0 0 0"/>
   </joint>
+  <!-- BASE — wide cylinder with top coupling disc -->
   <link name="base_link">
     <visual>
-      <geometry><cylinder length="0.1" radius="0.12"/></geometry>
-      <material name="dark_grey"/>
+      <origin xyz="0 0 0.05" rpy="0 0 0"/>
+      <geometry><cylinder length="0.10" radius="0.12"/></geometry>
+      <material name="c1"/>
+    </visual>
+    <visual>
+      <origin xyz="0 0 0.105" rpy="0 0 0"/>
+      <geometry><cylinder length="0.01" radius="0.10"/></geometry>
+      <material name="c1"/>
     </visual>
     <collision>
@@ -25,13 +36,23 @@
     <axis xyz="0 0 1"/>
   </joint>
+  <!-- SHOULDER — stacked disc / body / disc (Kuka style) -->
   <link name="shoulder_link">
     <visual>
-      <origin xyz="0 0 0.05" rpy="0 0 0"/>
-      <geometry><cylinder length="0.1" radius="0.08"/></geometry>
-      <material name="orange"/>
-    </visual>
-    <visual>
-      <geometry><sphere radius="0.065"/></geometry>
-      <material name="orange"/>
+      <!-- bottom coupling disc (joint_1 plane) -->
+      <origin xyz="0 0 0.012" rpy="0 0 0"/>
+      <geometry><cylinder length="0.024" radius="0.082"/></geometry>
+      <material name="c2"/>
+    </visual>
+    <visual>
+      <!-- shoulder body -->
+      <origin xyz="0 0 0.052" rpy="0 0 0"/>
+      <geometry><cylinder length="0.052" radius="0.068"/></geometry>
+      <material name="c2"/>
+    </visual>
+    <visual>
+      <!-- top coupling disc (joint_2 plane) -->
+      <origin xyz="0 0 0.088" rpy="0 0 0"/>
+      <geometry><cylinder length="0.024" radius="0.082"/></geometry>
+      <material name="c2"/>
     </visual>
     <collision>
@@ -47,13 +68,23 @@
     <limit lower="-1.57" upper="1.57" effort="50.0" velocity="1.0"/>
   </joint>
+  <!-- UPPER ARM — horizontal knuckle at joint_2, arm tube, knuckle at joint_3 end -->
   <link name="upper_arm">
     <visual>
-      <origin xyz="0 0 0.2" rpy="0 0 0"/>
-      <geometry><cylinder length="0.4" radius="0.055"/></geometry>
-      <material name="silver"/>
-    </visual>
-    <visual>
-      <geometry><sphere radius="0.06"/></geometry>
-      <material name="silver"/>
+      <!-- joint_2 horizontal knuckle (Y-axis pivot housing) -->
+      <origin xyz="0 0 0" rpy="1.5708 0 0"/>
+      <geometry><cylinder length="0.12" radius="0.068"/></geometry>
+      <material name="c3"/>
+    </visual>
+    <visual>
+      <!-- arm tube -->
+      <origin xyz="0 0 0.22" rpy="0 0 0"/>
+      <geometry><cylinder length="0.32" radius="0.048"/></geometry>
+      <material name="c3"/>
+    </visual>
+    <visual>
+      <!-- joint_3 horizontal knuckle at top end -->
+      <origin xyz="0 0 0.40" rpy="1.5708 0 0"/>
+      <geometry><cylinder length="0.10" radius="0.060"/></geometry>
+      <material name="c3"/>
     </visual>
     <collision>
@@ -69,13 +100,17 @@
     <limit lower="-2.0" upper="2.0" effort="30.0" velocity="1.5"/>
   </joint>
+  <!-- FOREARM — horizontal knuckle at joint_3, slim forearm tube -->
   <link name="forearm">
     <visual>
-      <origin xyz="0 0 0.15" rpy="0 0 0"/>
-      <geometry><cylinder length="0.3" radius="0.03"/></geometry>
-      <material name="orange"/>
-    </visual>
-    <visual>
-      <geometry><sphere radius="0.04"/></geometry>
-      <material name="orange"/>
+      <!-- joint_3 horizontal knuckle (Y-axis pivot housing) -->
+      <origin xyz="0 0 0" rpy="1.5708 0 0"/>
+      <geometry><cylinder length="0.09" radius="0.050"/></geometry>
+      <material name="c4"/>
+    </visual>
+    <visual>
+      <!-- forearm tube -->
+      <origin xyz="0 0 0.16" rpy="0 0 0"/>
+      <geometry><cylinder length="0.26" radius="0.028"/></geometry>
+      <material name="c4"/>
     </visual>
     <collision>
@@ -89,8 +124,15 @@
     <origin xyz="0 0 0.3" rpy="0 0 0"/>
   </joint>
+  <!-- WRIST + PALM -->
   <link name="gripper_base">
     <visual>
-      <geometry><box size="0.1 0.1 0.05"/></geometry>
-      <material name="dark_grey"/>
+      <origin xyz="0 0 -0.008" rpy="0 0 0"/>
+      <geometry><cylinder length="0.03" radius="0.038"/></geometry>
+      <material name="c5"/>
+    </visual>
+    <visual>
+      <origin xyz="0 0 0.013" rpy="0 0 0"/>
+      <geometry><box size="0.088 0.072 0.025"/></geometry>
+      <material name="c5"/>
     </visual>
     <collision>
@@ -105,8 +147,9 @@
     <limit lower="-0.04" upper="0.0" effort="10.0" velocity="0.1"/>
   </joint>
+  <!-- FINGERS -->
   <link name="left_finger">
     <visual>
       <geometry><box size="0.02 0.02 0.08"/></geometry>
-      <material name="silver"/>
+      <material name="c6"/>
     </visual>
     <collision>
@@ -125,5 +168,5 @@
     <visual>
       <geometry><box size="0.02 0.02 0.08"/></geometry>
-      <material name="silver"/>
+      <material name="c6"/>
     </visual>
     <collision>
